File: PWR_supply/12to5.sch (KiCad schematic (older format))
At the start: 3 parts, among them U2 LM7805CT

Commit message: PWR_supply labojumi veikti
Parts:
- C3: renamed from 0.1uF3; value CP1 -> 0.1uF
- C4: renamed from 0.1uF2; value CP1 -> 0.1uF
Changed lines of the file:
@@
 $Descr A4 11693 8268
 encoding utf-8
-Sheet 4 5
+Sheet 4 6
 Title ""
 Date ""
@@
 $EndComp
 $Comp
-L CP1 0.1uF2
+L CP1 C4
 U 1 1 58D252C4
 P 4500 2600
-F 0 "0.1uF2" H 4525 2700 50  0000 L CNN
-F 1 "CP1" H 4525 2500 50  0000 L CNN
+F 0 "C4" H 4525 2700 50  0000 L CNN
+F 1 "0.1uF" H 4525 2500 50  0000 L CNN
 F 2 "" H 4500 2600 50  0000 C CNN
 F 3 "" H 4500 2600 50  0000 C CNN
@@
 $EndComp
 $Comp
-L CP1 0.1uF3
+L CP1 C3
 U 1 1 58D252E3
 P 5800 2600
-F 0 "0.1uF3" H 5825 2700 50  0000 L CNN
-F 1 "CP1" H 5825 2500 50  0000 L CNN
+F 0 "C3" H 5825 2700 50  0000 L CNN
+F 1 "0.1uF" H 5825 2500 50  0000 L CNN
 F 2 "" H 5800 2600 50  0000 C CNN
 F 3 "" H 5800 2600 50  0000 C CNN
