File: PWR_supply/20VDC_to_3VDC.sch (KiCad schematic (older format))
At the start: 3 parts, among them U3 NCP1117DT33G

Commit message: PWR_supply labojumi veikti
Parts:
- C2: value 100uF -> 10uF
Changed lines of the file:
@@
 P 3600 2800
 F 0 "C2" H 3625 2900 50  0000 L CNN
-F 1 "100uF" H 3625 2700 50  0000 L CNN
+F 1 "10uF" H 3625 2700 50  0000 L CNN
 F 2 "" H 3600 2800 50  0000 C CNN
 F 3 "" H 3600 2800 50  0000 C CNN
