File: PWR_supply/3V.sch (KiCad schematic (older format))
At the start: 4 parts, among them U3 LM1117-3.3

Commit message: PWR_supply labojumi veikti
Parts:
- removed R1: 120R, symbol R
- removed U3: LM1117-3.3, symbol LM1117-3.3
- added U3: NCP1117DT33G, TO_SOT_Packages_SMD:TO-263-3Lead, symbol NCP1117DT33G
- C1: renamed from 10uF2; value CP1 -> 10uF
- C2: renamed from 100uF1; value CP1 -> 100uF
Connections:
- net 3.3Vout: now also U3.2 (VO)
- net GND: now also U3.1 (GND)
- net 5Vin renamed Vin
- net Vin: now also U3.3 (VI)
Changed lines of the file:
@@
 $Descr A4 11693 8268
 encoding utf-8
-Sheet 5 5
+Sheet 5 6
 Title ""
 Date ""
@@
 Comment4 ""
 $EndDescr
-$Comp
-L LM1117-3.3 U3
-U 1 1 58D259FF
-P 4200 2400
-F 0 "U3" H 4300 2150 50  0000 C CNN
-F 1 "LM1117-3.3" H 4200 2650 50  0000 C CNN
-F 2 "" H 4200 2400 50  0000 C CNN
-F 3 "" H 4200 2400 50  0000 C CNN
-	1    4200 2400
-	1    0    0    -1
-$EndComp
 Text HLabel 3200 2400 0    60   Output ~ 0
-5Vin
+Vin
 Text HLabel 4200 3150 3    60   Output ~ 0
 GND
@@
 	3900 2400 3200 2400
 $Comp
-L CP1 100uF1
+L CP1 C2
 U 1 1 58D25A4A
 P 3600 2800
-F 0 "100uF1" H 3625 2900 50  0000 L CNN
-F 1 "CP1" H 3625 2700 50  0000 L CNN
+F 0 "C2" H 3625 2900 50  0000 L CNN
+F 1 "100uF" H 3625 2700 50  0000 L CNN
 F 2 "" H 3600 2800 50  0000 C CNN
 F 3 "" H 3600 2800 50  0000 C CNN
@@
 $EndComp
 $Comp
-L CP1 10uF2
+L CP1 C1
 U 1 1 58D25A87
 P 4800 2800
-F 0 "10uF2" H 4825 2900 50  0000 L CNN
-F 1 "CP1" H 4825 2700 50  0000 L CNN
+F 0 "C1" H 4825 2900 50  0000 L CNN
+F 1 "10uF" H 4825 2700 50  0000 L CNN
 F 2 "" H 4800 2800 50  0000 C CNN
 F 3 "" H 4800 2800 50  0000 C CNN
@@
 Wire Wire Line
 	4200 2700 4200 3150
-$Comp
-L R R1
-U 1 1 58D6E8BE
-P 4600 2650
-F 0 "R1" V 4680 2650 50  0000 C CNN
-F 1 "120R" V 4600 2650 50  0000 C CNN
-F 2 "" V 4530 2650 50  0000 C CNN
-F 3 "" H 4600 2650 50  0000 C CNN
-	1    4600 2650
-	1    0    0    -1
-$EndComp
-Wire Wire Line
-	4600 2800 4600 2950
-Connection ~ 4600 2950
 Wire Wire Line
 	4500 2400 5300 2400
 Wire Wire Line
 	4800 2400 4800 2650
-Wire Wire Line
-	4600 2500 4600 2400
-Connection ~ 4600 2400
 Connection ~ 4800 2400
+$Comp
+L NCP1117DT33G U3
+U 1 1 58DC1701
+P 4200 2400
+F 0 "U3" H 4200 2625 50  0000 C CNN
+F 1 "NCP1117DT33G" H 4200 2550 50  0000 C CNN
+F 2 "TO_SOT_Packages_SMD:TO-263-3Lead" H 4250 2150 50  0001 L CNN
+F 3 "" H 4200 2400 50  0000 C CNN
+	1    4200 2400
+	1    0    0    -1
+$EndComp
 $EndSCHEMATC
