File: Battery/Battery.sch (KiCad schematic (older format))
At the start: 1 part

Commit message: pabeigts maajas darbs battery un iesaakts projekts controll unit
Parts:
- BT1: footprint battery:SMTU2032_footprint -> battery:502
Changed lines of the file:
@@
 F 0 "BT1" H 5550 3050 50  0000 L CNN
 F 1 "Battery_Cell" H 5550 2950 50  0000 L CNN
-F 2 "battery:SMTU2032_footprint" H 5450 3010 50  0001 C CNN
+F 2 "battery:502" H 5450 3010 50  0001 C CNN
 F 3 "" V 5450 3010 50  0000 C CNN
 	1    5450 2950
